File: kinx.brd (EAGLE design)
At the start: 122 x 86 mm, 45 parts, among them T1 MCP1825S

Commit message: fix silkscreen for power LED
Parts:
- renumbered P1 to LED_PWR
Changed lines of the file:
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@@
 <attribute name="VALUE" x="88.095" y="65.73" size="0.635" layer="26" ratio="10" rot="MR90"/>
 </element>
-<element name="R8" library="t32_ref" package="R0603" value="470R" x="68" y="36" rot="MR270">
+<element name="R8" library="t32_ref" package="R0603" value="470R" x="68" y="36" smashed="yes" rot="MR270">
 <attribute name="DESC" value="470R / 1 % /  0.1 W" x="-25" y="174" size="1.778" layer="28" rot="MR270" display="off"/>
 <attribute name="MF" value="Vishay" x="-25" y="174" size="1.778" layer="28" rot="MR270" display="off"/>
 <attribute name="MPN" value="CRCW0603470RFKEA" x="-25" y="174" size="1.778" layer="28" rot="MR270" display="off"/>
+<attribute name="NAME" x="68" y="36" size="0.7" layer="52" rot="MR0" align="center"/>
 <attribute name="OC_MOUSER" value="71-CRCW0603-470-E3" x="-25" y="174" size="1.778" layer="28" rot="MR270" display="off"/>
 <attribute name="PACKAGE" value="0603" x="-25" y="174" size="1.778" layer="28" rot="MR270" display="off"/>
 <attribute name="TYPE" value="Resistor" x="-25" y="174" size="1.778" layer="28" rot="MR270" display="off"/>
+<attribute name="VALUE" x="69.27" y="34.095" size="0.635" layer="26" ratio="10" rot="MR0"/>
 </element>
 <element name="R7" library="t32_ref" package="R0603" value="33R" x="85" y="67" smashed="yes" rot="MR0">
@@
 <attribute name="VALUE" x="42.809" y="69.99" size="0.889" layer="26" ratio="11" rot="MR0"/>
 </element>
-<element name="P1" library="t32_ref" package="LED-0805" value="" x="70.933" y="35.091" rot="MR90">
+<element name="LED_PWR" library="t32_ref" package="LED-0805" value="" x="70.933" y="35.091" rot="MR90">
 <attribute name="DESC" value="orange" x="-762.067" y="-187.909" size="1.778" layer="28" rot="MR90" display="off"/>
 <attribute name="MF" value="ROHM Semiconductor" x="-762.067" y="-187.909" size="1.778" layer="28" rot="MR90" display="off"/>
@@
 </signal>
 <signal name="N$41">
-<contactref element="P1" pad="+"/>
+<contactref element="LED_PWR" pad="+"/>
 <contactref element="U$1" pad="106"/>
 <wire x1="77.71" y1="38.04" x2="77.71" y2="36.71" width="0.2" layer="16"/>
@@
 <signal name="N$80">
 <contactref element="R8" pad="2"/>
-<contactref element="P1" pad="-"/>
+<contactref element="LED_PWR" pad="-"/>
 <wire x1="68.762" y1="36" x2="70.933" y2="35.98" width="0.4" layer="16"/>
 </signal>

Commit message: use 10K resistors to drive the LEDs
Parts:
- R1, R2, R3, R4: value (none) -> 10K
Changed lines of the file:
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@@
 <attribute name="VALUE" x="77.905" y="2.349" size="1.27" layer="27" ratio="10"/>
 </element>
-<element name="R1" library="rcl" package="R1206" value="" x="44" y="9" smashed="yes" rot="R90">
+<element name="R1" library="rcl" package="R1206" value="10K" x="44" y="9" smashed="yes" rot="R90">
 <attribute name="NAME" x="46.857" y="7.603" size="1.27" layer="25" rot="R90"/>
 <attribute name="VALUE" x="46.413" y="7.603" size="1.27" layer="27" rot="R90"/>
 </element>
-<element name="R2" library="rcl" package="R1206" value="" x="54" y="9" smashed="yes" rot="R90">
+<element name="R2" library="rcl" package="R1206" value="10K" x="54" y="9" smashed="yes" rot="R90">
 <attribute name="NAME" x="56.857" y="7.603" size="1.27" layer="25" rot="R90"/>
 <attribute name="VALUE" x="56.413" y="7.603" size="1.27" layer="27" rot="R90"/>
 </element>
-<element name="R3" library="rcl" package="R1206" value="" x="64" y="9" smashed="yes" rot="R90">
+<element name="R3" library="rcl" package="R1206" value="10K" x="64" y="9" smashed="yes" rot="R90">
 <attribute name="NAME" x="66.857" y="7.603" size="1.27" layer="25" rot="R90"/>
 <attribute name="VALUE" x="66.413" y="7.603" size="1.27" layer="27" rot="R90"/>
 </element>
-<element name="R4" library="rcl" package="R1206" value="" x="74" y="9" smashed="yes" rot="R90">
+<element name="R4" library="rcl" package="R1206" value="10K" x="74" y="9" smashed="yes" rot="R90">
 <attribute name="NAME" x="76.857" y="7.603" size="1.27" layer="25" rot="R90"/>
 <attribute name="VALUE" x="76.413" y="7.603" size="1.27" layer="27" rot="R90"/>
