File: kinx.sch (EAGLE design)
At the start: 45 parts, among them T1 MCP1825S

Commit message: Connect remaining VSS pins
Connections:
- net GND: now also U$1.USB1_VSS, U$1.VSS@3
Changed lines of the file:
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@@
 <part name="C13" library="t32_ref" deviceset="CAPACITOR-0.1UF" device="" value="0.1uF"/>
 <part name="GND37" library="t32_ref" deviceset="GND" device=""/>
+<part name="GND38" library="t32_ref" deviceset="GND" device=""/>
+<part name="GND39" library="t32_ref" deviceset="GND" device=""/>
 </parts>
 <sheets>
@@
 <instance part="C13" gate="G$1" x="-171.45" y="-15.24" rot="R90"/>
 <instance part="GND37" gate="1" x="-167.64" y="-15.24" rot="R90"/>
+<instance part="GND38" gate="1" x="-246.38" y="55.88" rot="R270"/>
+<instance part="GND39" gate="1" x="-246.38" y="40.64" rot="R270"/>
 </instances>
 <busses>
@@
 <wire x1="-294.64" y1="40.64" x2="-291.592" y2="40.64" width="0.1524" layer="91"/>
 </segment>
-</net>
+<segment>
+<pinref part="GND38" gate="1" pin="GND"/>
+<pinref part="U$1" gate="G$1" pin="VSS@3"/>
+<wire x1="-245.11" y1="55.88" x2="-241.3" y2="55.88" width="0.1524" layer="91"/>
+</segment>
+<segment>
+<pinref part="GND39" gate="1" pin="GND"/>
+<pinref part="U$1" gate="G$1" pin="USB1_VSS"/>
+<wire x1="-245.11" y1="40.64" x2="-241.3" y2="40.64" width="0.1524" layer="91"/>
+</segment>
+</net>

Commit message: Bugfix: wire up USB1_VBUS and all GND airwires
Connections:
- new net N$8: U$1.USB1_VBUS, USBHS.VBUS
Changed lines of the file:
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@@
+</segment>
+</net>
+<net name="N$8" class="0">
+<segment>
+<pinref part="USBHS" gate="G$1" pin="VBUS"/>
+<wire x1="-294.64" y1="30.48" x2="-259.08" y2="30.48" width="0.1524" layer="91"/>
+<wire x1="-259.08" y1="30.48" x2="-259.08" y2="33.02" width="0.1524" layer="91"/>
+<pinref part="U$1" gate="G$1" pin="USB1_VBUS"/>
+<wire x1="-259.08" y1="33.02" x2="-241.3" y2="33.02" width="0.1524" layer="91"/>
 </segment>
 </net>

Commit message: Switch to Molex 105133-0011 (USB 2.0 instead of USB)
Parts:
- USBFS, USBHS: DIGIKEY WM9734CT-ND -> WM10134CT-ND
Changed lines of the file:
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@@
 <part name="GND12" library="t32_ref" deviceset="GND" device=""/>
 <part name="USBFS" library="molex-105133-0001" deviceset="105133-0001" device="">
-<attribute name="DIGIKEY" value="WM9734CT-ND"/>
+<attribute name="DIGIKEY" value="WM10134CT-ND"/>
 <attribute name="OC_MOUSER" value="538-105133-0001"/>
 </part>
 <part name="USBHS" library="molex-105133-0001" deviceset="105133-0001" device="">
-<attribute name="DIGIKEY" value="WM9734CT-ND"/>
+<attribute name="DIGIKEY" value="WM10134CT-ND"/>
 <attribute name="OC_MOUSER" value="538-105133-0001"/>
 </part>
